Commit message: make base_link simple without inertial

File: rs_series_description/urdf/rs007l.urdf.xacro (robot description, xacro)
@@ -57,6 +57,13 @@
         </inertial>
     </xacro:macro>
+    <!-- !The root link base_link has an inertia specified in the URDF, but KDL does not support a
+    root link with an inertia.  As a workaround, you can add an extra dummy link to your URDF. -->
+    <link name="base_link" />
+    <joint name="joint0" type="fixed">
+        <parent link="base_link" />
+        <child link="link0" />
+    </joint>
     <!-- Link 0 -->
-    <link name="base_link">
+    <link name="link0">
         <visual>
             <geometry>
@@ -82,5 +89,5 @@
             velocity="${j1_velocity_limit}" />
         <origin xyz="0 0 ${j0_length}" rpy="0 0 0" />
-        <parent link="base_link" />
+        <parent link="link0" />
         <child link="link1" />
         <dynamics damping="0.0" friction="0.0" />

Commit message: replace collision into simple geometry

File: rs_series_description/urdf/rs007l.urdf.xacro (robot description, xacro)
@@ -76,8 +76,10 @@
             <geometry>
                 <!-- TODO replace collision mesh into *.dae for lower computation cost -->
-                <mesh filename="package://rs_series_description/meshes/visual/rs007l/RS007L_J0.stl" />
-            </geometry>
-            <material name="White" />
-            <origin rpy="0 0 0" xyz="0 0 0" />
+                <box size="0.2 0.25 0.2" />
+                <!-- <mesh
+                filename="package://rs_series_description/meshes/visual/rs007l/RS007L_J0.stl" /> -->
+            </geometry>
+            <material name="White" />
+            <origin xyz="0.0 0.0 0.1" rpy="0.0 0.0 0.0" />
         </collision>
         <xacro:default_inertial mass="${j0_mass}" />
@@ -104,8 +106,10 @@
             <geometry>
                 <!-- TODO replace collision mesh into *.dae for lower computation cost -->
-                <mesh filename="package://rs_series_description/meshes/visual/rs007l/RS007L_J1.stl" />
-            </geometry>
-            <material name="White" />
-            <origin rpy="0 0 0" xyz="0 0 0" />
+                <box size="0.25 0.25 0.25" />
+                <!-- <mesh
+                filename="package://rs_series_description/meshes/visual/rs007l/RS007L_J1.stl" /> -->
+            </geometry>
+            <material name="White" />
+            <origin rpy="0 0 0" xyz="0 0 -0.05" />
         </collision>
         <xacro:default_inertial mass="${j1_mass}" />
@@ -132,8 +136,10 @@
             <geometry>
                 <!-- TODO replace collision mesh into *.dae for lower computation cost -->
-                <mesh filename="package://rs_series_description/meshes/visual/rs007l/RS007L_J2.stl" />
-            </geometry>
-            <material name="White" />
-            <origin xyz="0 0 0" rpy="0 ${dh_j1_j2_roty*-1} 0" />
+                <box size="0.2 0.2 0.6" />
+                <!-- <mesh
+                filename="package://rs_series_description/meshes/visual/rs007l/RS007L_J2.stl" /> -->
+            </geometry>
+            <material name="White" />
+            <origin xyz="0.25 0 -0.1" rpy="0 ${dh_j1_j2_roty*-1} 0" />
         </collision>
         <xacro:default_inertial mass="0${j2_mass}" />
@@ -160,5 +166,7 @@
             <geometry>
                 <!-- TODO replace collision mesh into *.dae for lower computation cost -->
-                <mesh filename="package://rs_series_description/meshes/visual/rs007l/RS007L_J3.stl" />
+                <box size="0.2 0.2 0.2" />
+                <!-- <mesh
+                filename="package://rs_series_description/meshes/visual/rs007l/RS007L_J3.stl" /> -->
             </geometry>
             <material name="White" />
@@ -188,8 +196,10 @@
             <geometry>
                 <!-- TODO replace collision mesh into *.dae for lower computation cost -->
-                <mesh filename="package://rs_series_description/meshes/visual/rs007l/RS007L_J4.stl" />
-            </geometry>
-            <material name="White" />
-            <origin xyz="0 0 ${j4_length}" rpy="0 0 0" />
+                <box size="0.15 0.15 0.4" />
+                <!-- <mesh
+                filename="package://rs_series_description/meshes/visual/rs007l/RS007L_J4.stl" /> -->
+            </geometry>
+            <material name="White" />
+            <origin xyz="0 0 ${j4_length-0.2}" rpy="0 0 0" />
         </collision>
         <xacro:default_inertial mass="${j4_mass}" />
@@ -216,8 +226,10 @@
             <geometry>
                 <!-- TODO replace collision mesh into *.dae for lower computation cost -->
-                <mesh filename="package://rs_series_description/meshes/visual/rs007l/RS007L_J5.stl" />
-            </geometry>
-            <material name="White" />
-            <origin xyz="0 0 0" rpy="0 ${dh_j4_j5_roty*-1} 0" />
+                <box size="0.1 0.1 0.1" />
+                <!-- <mesh
+                filename="package://rs_series_description/meshes/visual/rs007l/RS007L_J5.stl" /> -->
+            </geometry>
+            <material name="White" />
+            <origin xyz="0.05 0 0" rpy="0 ${dh_j4_j5_roty*-1} 0" />
         </collision>
         <xacro:default_inertial mass="${j5_mass}" />
@@ -244,5 +256,7 @@
             <geometry>
                 <!-- TODO replace collision mesh into *.dae for lower computation cost -->
-                <mesh filename="package://rs_series_description/meshes/visual/rs007l/RS007L_J6.stl" />
+                <cylinder radius="0.02" length="0.005" />
+                <!-- <mesh
+                filename="package://rs_series_description/meshes/visual/rs007l/RS007L_J6.stl" /> -->
             </geometry>
             <material name="Black" />
